File: output/pcbs/Keiler.kicad_pcb (KiCad board)
At the start: 2 copper layers, 133.9 x 103.2 mm, 44 parts

Commit message: Nicer routing
Parts:
- moved S27 2.15 mm to (156.3, 99.1)
- moved S9 2.15 mm to (156.3, 99.1)
- moved _5 2.15 mm to (140.7, 169.4)
- moved S15 2.15 mm to (201.3, 113.9)
- moved S16 2.15 mm to (186.0, 167.7)
- moved S17 2.15 mm to (205.7, 171.5)
- moved S33 2.15 mm to (201.3, 113.9)
- moved S34 2.15 mm to (186.0, 167.7)
- moved S35 2.15 mm to (205.7, 171.5)
- moved S23 2.15 mm to (139.8, 123.7)
- moved S5 2.15 mm to (139.8, 123.7)
- moved S22 2.15 mm to (143.1, 140.4)
- moved S25 2.15 mm to (161.0, 132.7)
- moved S4 2.15 mm to (143.1, 140.4)
- moved S7 2.15 mm to (161.0, 132.7)
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Routing:
- net P4: track 99.6 -> 104.4 mm
- net P3: track 118.1 -> 122.6 mm
- net P5: track 82.2 -> 86.6 mm
- net P9: track 157.4 -> 161.5 mm
- net P6: track 145.2 -> 149.2 mm
- net P7: track 126.7 -> 130.8 mm
- net RST: track 42.1 -> 46.2 mm
- net P16: track 147.0 -> 143.7 mm
- net GND: track 899.4 -> 902.5 mm
- net P8: track 111.4 -> 109.3 mm
- net P15: track 169.3 -> 168.3 mm
- net P21: track 89.0 -> 89.9 mm
- net P19: track 117.1 -> 118.0 mm
- net pos: track 17.7 -> 17.0 mm

Commit message: Nicer routing
Parts:
- moved S16 4.00 mm to (182.4, 169.6)
- moved S34 4.00 mm to (182.4, 169.6)
- moved S15 4.00 mm to (197.7, 115.8)
- moved S33 4.00 mm to (197.7, 115.8)
- moved _7 4.00 mm to (167.0, 109.9)
- moved S27 4.00 mm to (152.7, 100.9)
- moved S9 4.00 mm to (152.7, 100.9)
- moved MCU1 4.00 mm to (217.7, 146.9)
- moved S22 4.00 mm to (139.6, 142.3)
- moved S4 4.00 mm to (139.6, 142.3)
- moved S21 4.00 mm to (112.7, 131.1)
- moved S3 4.00 mm to (112.7, 131.1)
- moved S17 4.00 mm to (202.2, 173.3)
- moved S35 4.00 mm to (202.2, 173.3)
- moved S1 4.00 mm to (125.1, 162.7)
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Routing:
- net GND: track 902.5 -> 919.7 mm
- net P19: track 118.0 -> 118.7 mm
